File: KiCad/LPF_HF+6.kicad_pcb (KiCad board)
At the start: 2 copper layers, 250 x 160 mm, 134 parts, among them J1 Conn_01x07, J2 12V INPUT, J3 RF input, J4 Conn_01x07, J5 RF output, U1 AMS1117-5, U2 74AHC595, U3 ULN2003

Commit message: ERC DRC run and show no significant issues
Parts:
- removed the C39 at (332.1, 92.4)
- removed REF** (x2): OSHW-Logo2_24.3x20mm_SilkScreen, Symbol:OSHW-Logo2_24.3x20mm_SilkScreen
- J3: value RF input -> LFP_IN
- L18, L19: footprint Custom_Ferrites_FT:T94-SWR_TRAFO -> LPF_Footprints:T94-SWR_TRAFO
Routing:
- net +12V: track 718.6 -> 710.4 mm
- net /40-30m_REL: track 433.5 -> 429.3 mm
- net GND: track 103.5 -> 99.6 mm, vias 1018 -> 1017
- net /80m_REL: track 404.2 -> 400.3 mm
- net +5V: track 55.7 -> 52.5 mm
- net /160m_REL: track 374.2 -> 371.6 mm
- net /20-17m: track 462.8 -> 460.3 mm
- net /15-10m_REL: track 491.5 -> 489.5 mm
- net /6m_REL: track 521.1 -> 519.5 mm
- net /LPF_OUT: track 93.5 -> 92.3 mm
- net PWR_FWD: track 28.6 -> 27.8 mm
- net Net-(D20-A): track 53.7 -> 53.0 mm
- net Net-(J4-Pin_7): track 24.6 -> 23.9 mm
- net Net-(J4-Pin_1): track 19.1 -> 18.5 mm
- net Net-(J4-Pin_2): track 17.3 -> 16.8 mm
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